File: Analog Light Intensity Meter/Analog Light Intensity Meter.kicad_pcb (KiCad board)
At the start: 2 copper layers, 75 x 105 mm, 37 parts, among them J1 Conn_01x02, U1 LM324, U2 LM324, U3 LM324

Commit message: V1
Parts:
- D1, D10, D2, D3, D4, D5, D6, D7, D8, D9, R1, R11, R3, R5, R7, R9: moved to F.Cu
