File: Analog Light Intensity Meter/Analog Light Intensity Meter.kicad_sch (KiCad schematic)
At the start: 37 parts, among them J1 Conn_01x02, U1 LM324, U2 LM324, U3 LM324

Commit message: V1
Other:
- moved on the sheet: D1, D10, D2, D3, D4, D5, D6, D7, D8, D9, J1, R1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
